Commit message: new training new urdf

File: URDF_FILES/6dof/urdf/gen3_6dof.urdf (robot description, URDF)
Before this commit: robot gen3, 13 links, 12 joints
Links:
- link base_link: geometry collision mesh filename=../meshes/base_link.STL; visual mesh filename=../meshes/base_link.STL
- link bicep_link: geometry collision mesh filename=../meshes/bicep_link.STL; visual mesh filename=../meshes/bicep_link.STL
- link bracelet_link: geometry collision mesh filename=../meshes/bracelet_with_vision_link.STL; visual mesh filename=../meshes/bracelet_with_vision_link.STL
- link forearm_link: geometry collision mesh filename=../meshes/forearm_link.STL; visual mesh filename=../meshes/forearm_link.STL
- link shoulder_link: geometry collision mesh filename=../meshes/shoulder_link.STL; visual mesh filename=../meshes/shoulder_link.STL
- link spherical_wrist_1_link: geometry collision mesh filename=../meshes/spherical_wrist_1_link.STL; visual mesh filename=../meshes/spherical_wrist_1_link.STL
- link spherical_wrist_2_link: geometry collision mesh filename=../meshes/spherical_wrist_2_link.STL; visual mesh filename=../meshes/spherical_wrist_2_link.STL

Commit message: new urdf policy

File: URDF_FILES/6dof/urdf/gen3_6dof.urdf (robot description, URDF)
Before this commit: robot gen3, 13 links, 12 joints
Joints:
- joint end_effector: origin xyz=0 0 -0.0615250000000001 rpy=3.14159265358979 1.09937075168372E-32 3.14159265358979 -> xyz=0 0 -0.0615250000000001 rpy=0 0 0
